Commit message: Local Costmap Finally working for 2D Obstacle layer and racecar model, update to 3D voxel and truck

File: nav2_bringup/bringup/urdf/ackerman.urdf (robot description, URDF)
Before this commit: robot ackermann_robot, 13 links, 12 joints
Links:
- link base_footprint: geometry 
- link base_link: mass 10 -> 5

File: nav2_bringup/bringup/urdf/ackerman.xacro (robot description, xacro)
@@ -65,7 +65,7 @@
   </material>
     <!--Robot Footprint -->
-  <!-- <link name="base_footprint"/> -->
+  <link name="base_footprint"/>
   <!--Robot Footprint Visualization-->
-  <link name="base_footprint">
+  <!-- <link name="base_footprint">
     <visual>
       <origin xyz="0 0 0" rpy="0 0 0"/>
@@ -75,5 +75,5 @@
       <material name="red"/>
     </visual>
-  </link>
+  </link> -->
   <!-- Base Link -->
   <link name="base_link">
@@ -91,5 +91,5 @@
       </geometry>
     </collision>
-    <xacro:box_inertia m="10" w="${base_width}" d="${base_length}" h="${base_height}"/>
+    <xacro:box_inertia m="5" w="${base_width}" d="${base_length}" h="${base_height}"/>
   </link>
   <joint name="base_joint" type = "fixed">
@@ -453,5 +453,5 @@
       </ros>
       <!-- further reduced the update rate -->
-      <update_rate>1.0</update_rate>
+      <update_rate>30</update_rate>
       <!-- wheels -->
       <front_left_joint>frontal_wheel_left_frontal_joint</front_left_joint>

File: nav2_bringup/bringup/urdf/sam_bot.urdf (robot description, URDF)
Before this commit: robot sam_bot, 16 links, 15 joints
Links:
- removed link first_shaft_horizontal_shaft_link
- removed link first_wheel_left_link
- removed link first_wheel_right_link
- removed link fourth_shaft_horizontal_shaft_link
- removed link fourth_wheel_left_link
- removed link fourth_wheel_right_link
- removed link front_left_steering_link
- removed link front_right_steering_link
- removed link second_shaft_horizontal_shaft_link
- removed link second_wheel_left_link
- removed link second_wheel_right_link
- removed link third_shaft_horizontal_shaft_link
- removed link third_wheel_left_link
- removed link third_wheel_right_link
- added link camera_depth_frame
- added link camera_link, mass 0.035; collision box size=0.015 0.130 0.022; visual box size=0.015 0.130 0.022
- added link drivewhl_l_link, mass 0.5; collision cylinder length=0.04 radius=0.1; visual cylinder length=0.04 radius=0.1
- added link drivewhl_r_link, mass 0.5; collision cylinder length=0.04 radius=0.1; visual cylinder length=0.04 radius=0.1
- added link front_caster, mass 0.5; collision sphere radius=0.060000000000000026; visual sphere radius=0.060000000000000026
- added link imu_link, mass 0.1; collision box size=0.1 0.1 0.1; visual box size=0.1 0.1 0.1
- added link lidar_link, mass 0.125; collision cylinder length=0.055 radius=0.0508; visual cylinder length=0.055 radius=0.0508
- link base_footprint: mass None -> 0
- link base_link: mass 500 -> 15; geometry collision box size=0.42 0.31 0.18; visual box size=0.42 0.31 0.18
Joints:
- removed joint first_shaft_horizontal_shaft_joint
- removed joint first_wheel_left_joint
- removed joint first_wheel_right_joint
- removed joint fourth_shaft_horizontal_shaft_joint
- removed joint fourth_wheel_left_joint
- removed joint fourth_wheel_right_joint
- removed joint front_left_steer_joint
- removed joint front_right_steer_joint
- removed joint second_shaft_horizontal_shaft_joint
- removed joint second_wheel_left_joint
- removed joint second_wheel_right_joint
- removed joint third_shaft_horizontal_shaft_joint
- removed joint third_wheel_left_joint
- removed joint third_wheel_right_joint
- added joint camera_depth_joint: type fixed, parent camera_link, child camera_depth_frame, origin xyz=0 0 0 rpy=-1.5707963267948966 0 -1.5707963267948966
- added joint camera_joint: type fixed, parent base_link, child camera_link, origin xyz=0.215 0 0.05 rpy=0 0 0
- added joint caster_joint: type fixed, parent base_link, child front_caster, origin xyz=0.14 0.0 -0.09 rpy=0 0 0
- added joint drivewhl_l_joint: type continuous, parent base_link, child drivewhl_l_link, origin xyz=-0.12 0.18 -0.05 rpy=0 0 0, axis 0 1 0
- added joint drivewhl_r_joint: type continuous, parent base_link, child drivewhl_r_link, origin xyz=-0.12 -0.18 -0.05 rpy=0 0 0, axis 0 1 0
- added joint imu_joint: type fixed, parent base_link, child imu_link, origin xyz=0 0 0.01
- added joint lidar_joint: type fixed, parent base_link, child lidar_link, origin xyz=0 0 0.12 rpy=0 0 0
- joint base_joint: child base_footprint -> base_link; origin xyz=0.0 0.0 -0.877 rpy=0 0 0 -> xyz=0.0 0.0 0.15000000000000002 rpy=0 0 0; parent base_link -> base_footprint

File: nav2_bringup/bringup/urdf/sam_bot.xacro (robot description, xacro)
@@ -1,57 +1,15 @@
 <?xml version="1.0"?>
 <robot name="sam_bot" xmlns:xacro="http://ros.org/wiki/xacro">
-    <!-- Material Definitions -->
-<!-- Init colour -->
-  <material name="black">
-      <color rgba="0.0 0.0 0.0 1.0"/>
-  </material>
-  <material name="dark">
-    <color rgba="0.3 0.3 0.3 1.0"/>
-  </material>
-  <material name="light_black">
-    <color rgba="0.4 0.4 0.4 1.0"/>
-  </material>
-  <material name="blue">
-    <color rgba="0.0 0.0 0.8 1.0"/>
-  </material>
-  <material name="green">
-    <color rgba="0.0 0.8 0.0 1.0"/>
-  </material>
-  <material name="grey">
-    <color rgba="0.5 0.5 0.5 1.0"/>
-  </material>
-  <material name="orange">
-    <color rgba="1.0 0.4235 0.0392 1.0"/>
-  </material>
-  <material name="brown">
-    <color rgba="0.8706 0.8118 0.7647 1.0"/>
-  </material>
-  <material name="red">
-    <color rgba="0.8 0.0 0.0 1.0"/>
-  </material>
-  <material name="white">
-    <color rgba="1.0 1.0 1.0 1.0"/>
-  </material>
   <!-- Define robot constants -->
-  <xacro:property name="base_width" value="2.548"/>
-  <xacro:property name="base_length" value="9.605"/>
-  <xacro:property name="base_height" value="0.877"/> <!-- Calculado na mão-->
-  <xacro:property name="wheel_mass" value="74"/> <!-- given by manual: https://jipco.com.sa/wp-content/uploads/2020/11/Arocs_4542_B_51_Std.pdf-->
-  <xacro:property name="wheel_radius" value="0.536"/> <!-- given by manual: https://jipco.com.sa/wp-content/uploads/2020/11/Arocs_4542_B_51_Std.pdf-->
-  <!-- webiste converter Michelin: https://tire-calc.com/pt/comparison/385-65-r22.5-and-385-55-r22.5/-->
-  <xacro:property name="wheel_width" value="0.385"/>
+  <xacro:property name="base_width" value="0.31"/>
+  <xacro:property name="base_length" value="0.42"/>
+  <xacro:property name="base_height" value="0.18"/>
+  <xacro:property name="wheel_radius" value="0.10"/>
+  <xacro:property name="wheel_width" value="0.04"/>
   <xacro:property name="wheel_ygap" value="0.025"/>
-  <xacro:property name="wheel_zoff" value="0.341"/> <!-- Calculado na mão-->
-  <xacro:property name="wheel_xoff" value="3.302"/> <!-- First shaft, Frontal-->
-  <xacro:property name="wheel2_xoff" value="1.552"/> <!-- Second Shaft, Frontal-->
-  <xacro:property name="wheel3_xoff" value="-2.152"/> <!-- Third Shaft, Rear -->
-  <xacro:property name="wheel4_xoff" value="-3.502"/> <!-- Fourth Shaft, Rear -->
-  <!-- Define the frontal shaft bar size-->
-  <xacro:property name="steering_bar_radius" value="0.0536"/>
-  <xacro:property name="steering_bar_length" value="2.548"/>
-  <!-- Define axles properties for the steering wheels (frontal)-->
-  <xacro:property name="axle_length" value="0.5"/>
-  <xacro:property name="axle_radius" value="0.25"/>
-      <!-- Define inertial property macros -->
+  <xacro:property name="wheel_zoff" value="0.05"/>
+  <xacro:property name="wheel_xoff" value="0.12"/>
+  <xacro:property name="caster_xoff" value="0.14"/>
+  <!-- Define some commonly used intertial properties  -->
   <xacro:macro name="box_inertia" params="m w h d">
     <inertial>
@@ -63,10 +21,16 @@
   <xacro:macro name="cylinder_inertia" params="m r h">
     <inertial>
-     <origin xyz="0 0 0" rpy="0 0 0"/>
-     <mass value="${m}"/>
-     <inertia ixx="${(m/12) * (3*r*r + h*h)}" ixy="0.0" ixz="0.0" iyy="${(m/12) * (3*r*r + h*h)}" iyz="0.0" izz="${(m/2) * r*r}"/>
+      <origin xyz="0 0 0" rpy="${pi/2} 0 0" />
+      <mass value="${m}"/>
+      <inertia ixx="${(m/12) * (3*r*r + h*h)}" ixy = "0" ixz = "0" iyy="${(m/12) * (3*r*r + h*h)}" iyz = "0" izz="${(m/2) * (r*r)}"/>
     </inertial>
   </xacro:macro>
-    <!-- Robot Base -->
+  <xacro:macro name="sphere_inertia" params="m r">
+    <inertial>
+      <mass value="${m}"/>
+      <inertia ixx="${(2/5) * m * (r*r)}" ixy="0.0" ixz="0.0" iyy="${(2/5) * m * (r*r)}" iyz="0.0" izz="${(2/5) * m * (r*r)}"/>
+    </inertial>
+  </xacro:macro>
+  <!-- Robot Base -->
   <link name="base_link">
     <visual>
@@ -78,228 +42,316 @@
       </material>
     </visual>
-    <xacro:box_inertia m="500" w="${base_width}" d="${base_length}" h="${base_height}"/>
-  </link>
-    <!-- Robot Footprint -->
-  <link name="base_footprint"/>
-<!--Robot Footprint Visualization-->
-  <!-- <link name="base_footprint">
-    <visual>
-      <origin xyz="0 0 0" rpy="0 0 0"/>
-      <geometry>
-        <box size="${base_length} ${base_width} 0.001"/>
-      </geometry>
-      <material name="red"/>
-    </visual>
-  </link>  -->
+    <collision>
+      <geometry>
+        <box size="${base_length} ${base_width} ${base_height}"/>
+      </geometry>
+    </collision>
+    <xacro:box_inertia m="15" w="${base_width}" d="${base_length}" h="${base_height}"/>
+  </link>
+   <!-- Robot Footprint -->
+  <link name="base_footprint">
+  	<xacro:box_inertia m="0" w="0" d="0" h="0"/>
+  </link>
   <joint name="base_joint" type="fixed">
-    <parent link="base_link"/>
-    <child link="base_footprint"/>
-    <origin xyz="0.0 0.0 ${-(wheel_radius+wheel_zoff)}" rpy="0 0 0"/>
-  </joint>
-   <!-- Bar Definition -->
-  <xacro:macro name="horizontal_shaft" params="xpos ypos prefix_name ">
-    <link name="${prefix_name}_horizontal_shaft_link">
+    <parent link="base_footprint"/>
+    <child link="base_link"/>
+    <origin xyz="0.0 0.0 ${(wheel_radius+wheel_zoff)}" rpy="0 0 0"/>
+  </joint>
+  <!-- Wheels -->
+  <xacro:macro name="wheel" params="prefix x_reflect y_reflect">
+    <link name="${prefix}_link">
       <visual>
+        <origin xyz="0 0 0" rpy="${pi/2} 0 0"/>
         <geometry>
-          <cylinder radius="${steering_bar_radius}" length="${steering_bar_length + wheel_ygap}"/>
+            <cylinder radius="${wheel_radius}" length="${wheel_width}"/>
         </geometry>
-        <material name="green">
+        <material name="Gray">
+          <color rgba="0.5 0.5 0.5 1.0"/>
         </material>
-        <origin xyz="0 0 0" rpy="0 ${pi/2} 0"/>
       </visual>
       <collision>
+        <origin xyz="0 0 0" rpy="${pi/2} 0 0"/>
         <geometry>
-          <cylinder radius="${steering_bar_radius}" length="${steering_bar_length}"/>
+          <cylinder radius="${wheel_radius}" length="${wheel_width}"/>
         </geometry>
-        <origin xyz="0 0 0" rpy="0 ${pi/2} 0"/>
       </collision>
-      <xacro:cylinder_inertia m="1" r="${steering_bar_radius}" h="${steering_bar_length}"/>
+      <xacro:cylinder_inertia m="0.5" r="${wheel_radius}" h="${wheel_width}"/>
     </link>
-  </xacro:macro>
-    <!-- Horizontal shafts instances -->
-  <xacro:horizontal_shaft xpos="0" ypos="0" prefix_name="first_shaft" />
-  <xacro:horizontal_shaft xpos="0" ypos="0" prefix_name="second_shaft" />
-  <xacro:horizontal_shaft xpos="0" ypos="0" prefix_name="third_shaft" />
-  <xacro:horizontal_shaft xpos="0" ypos="0" prefix_name="fourth_shaft" />
-    <!-- Horizontal shaft to base link connection -->
-  <xacro:macro name="horizontal_shaft_joint" params="prefix_name xpos ypos">
-    <joint name="${prefix_name}_horizontal_shaft_joint" type="fixed">
+    <joint name="${prefix}_joint" type="continuous">
       <parent link="base_link"/>
-      <child link="${prefix_name}_horizontal_shaft_link"/>
-      <origin xyz="${xpos} ${ypos} ${-wheel_zoff}" rpy="0 0 ${pi/2}"/>
-      <axis xyz="0 0 1"/>
-      <!-- <limit lower="-0.131" upper="0.131" effort="10000000" velocity="1000000"/> --> <!-- Just if change to revolute joint-->
+      <child link="${prefix}_link"/>
+      <origin xyz="${x_reflect*wheel_xoff} ${y_reflect*(base_width/2+wheel_ygap)} ${-wheel_zoff}" rpy="0 0 0"/>
+      <axis xyz="0 1 0"/>
     </joint>
   </xacro:macro>
-  <xacro:horizontal_shaft_joint prefix_name="first_shaft" xpos="${wheel_xoff}" ypos="0" />
-  <xacro:horizontal_shaft_joint prefix_name="second_shaft" xpos="${wheel2_xoff}" ypos="0" />
-  <xacro:horizontal_shaft_joint prefix_name="third_shaft" xpos="${wheel3_xoff}" ypos="0" />
-  <xacro:horizontal_shaft_joint prefix_name="fourth_shaft" xpos="${wheel4_xoff}" ypos="0" />
-    <!-- Define Steering Axle Links -->
-  <xacro:macro name="steer" params="prefix xpos ypos">
-    <link name="${prefix}_steering_link">
-      <visual>
-        <geometry>
-          <cylinder radius="${axle_radius}" length="${axle_length}"/>
-        </geometry>
-        <material name="white"/>
-      </visual>
-      <collision>
-        <geometry>
-          <cylinder radius="${axle_radius}" length="${axle_length}"/>
-        </geometry>
-      </collision>
-      <xacro:cylinder_inertia m="2" r="${axle_radius}" h="${axle_length}"/>
-    </link>
-  </xacro:macro>
-  <!-- The Creation of the Steering Links must come before the joints definition, otherwise Rviz will show TF error-->
-  <xacro:steer prefix="front_right" xpos="${-0.0001}" ypos="${0.0001}" />
-  <xacro:steer prefix="front_left" xpos="${-0.0001}" ypos="${-0.0001}" />
-    <!-- Define Steer Joint Macros-->
-  <xacro:macro name="steer_joint" params="prefix xpos ypos">
-    <joint name="${prefix}_steer_joint" type="revolute">
-      <parent link="first_shaft_horizontal_shaft_link" />
-      <child link="${prefix}_steering_link" />
-      <origin xyz="${xpos} ${ypos} ${-0.001}" rpy="0 0 0" />
-      <axis xyz="0 0 1" />
-      <limit lower="-0.524" upper="0.524" effort="10000000" velocity="1000000" />
-    </joint>
-  </xacro:macro>
-  <xacro:steer_joint prefix="front_left" xpos="${base_width/2 + wheel_ygap}" ypos="0" />
-  <xacro:steer_joint prefix="front_right" xpos="-${base_width/2 + wheel_ygap}" ypos="0" />
-    <!-- Wheels -->
-  <xacro:macro name="wheel" params="prefix xpos ypos wheel_num">
-      <!-- calculate moments of inertia -->
-      <xacro:property name="wheel_mass" value="74"/>
-      <xacro:property name="wheel_radius" value="0.536"/>
-      <xacro:property name="ixx_iyy_inertia" value="0.5 * ${wheel_mass} * ${wheel_radius} * ${wheel_radius}"/>
-      <xacro:property name="izz_inertia" value="${wheel_mass} * ${wheel_radius} * ${wheel_radius}"/>
-      <link name="${prefix}_link">
-        <visual>
-          <origin xyz="0 0 0" rpy="${pi/2} 0 0"/>
-          <geometry>
-              <cylinder radius="${wheel_radius}" length="${wheel_width}"/>
-          </geometry>
-          <material name="Gray">
-            <color rgba="0.5 0.5 0.5 1.0"/>
-          </material>
-        </visual>
-        <!-- Add mass and inertia -->
-              <!-- Add mass and inertia -->
-        <inertial>
-          <origin xyz="0 0 0" rpy="0 0 0"/>
-          <mass value="${wheel_mass}"/>
-          <inertia ixx="${ixx_iyy_inertia}" ixy="0" ixz="0" iyy="${ixx_iyy_inertia}" iyz="0" izz="${izz_inertia}"/>
-        </inertial>
-        <collision>
-          <geometry>
-            <cylinder radius="${wheel_radius}" length="${wheel_width}"/>
-          </geometry>
-          <origin xyz="0 0 0" rpy="${pi/2} 0 0"/>
-          <xacro:if value="${wheel_num == 1 or wheel_num == 4}">
-              <surface>
-                <friction>
-                  <ode>
-                    <mu>1.0</mu>
-                    <mu2>1.0</mu2>
-                    <kp>5000000.0</kp>
-                    <kd>1.0</kd>
-                    <fdir1>1 0 0</fdir1>
-                    <slip1>0.0</slip1>
-                    <slip2>0.0</slip2>
-                  </ode>
-                </friction>
-              </surface>
-          </xacro:if>
-          <xacro:unless value="${wheel_num == 1 or wheel_num == 4}">
-              <surface>
-                <friction>
-                  <ode>
-                    <mu>0.2</mu>
-                    <mu2>0.2</mu2>
-                    <kp>1000000.0</kp>
-                    <kd>0.5</kd>
-                    <fdir1>1 0 0</fdir1>
-                    <slip1>0.0</slip1>
-                    <slip2>0.0</slip2>
-                  </ode>
-                </friction>
-              </surface>
-          </xacro:unless>
-        </collision>
-        <xacro:cylinder_inertia m="${wheel_mass}" r="${wheel_radius}" h="${wheel_width}"/>
-      </link>
-      <!-- condition to check which wheel is being instantiated -->
-      <xacro:if value="${wheel_num == 1 or wheel_num == 4}">
-        <!-- First and fourth wheels are continuous and children of the steering joints/base link -->
-        <joint name="${prefix}_joint" type="continuous">
-          <xacro:if value="${prefix == 'first_wheel_left' or prefix == 'first_wheel_right'}">
-            <parent link="front_${prefix[12:]}_steering_link"/>
-            <origin xyz="${xpos} ${ypos} 0" rpy="0 0 1.57"/>
-          </xacro:if>
-          <xacro:unless value="${prefix == 'first_wheel_left' or prefix == 'first_wheel_right'}">
-            <parent link="fourth_shaft_horizontal_shaft_link"/>
-            <origin xyz="${xpos} ${ypos} ${0}" rpy="0 0 1.57"/>
-          </xacro:unless>
-          <child link="${prefix}_link"/>
-          <axis xyz="0 -1 0"/>
-        </joint>
-      </xacro:if>
-      <xacro:unless value="${wheel_num == 1 or wheel_num == 4}">
-          <!-- Second and third wheels are fixed type and children of respective shafts -->
-        <joint name="${prefix}_joint" type="fixed">
-          <parent link="${'second' if 'second' in prefix else 'third'}_shaft_horizontal_shaft_link"/>
-          <child link="${prefix}_link"/>
-          <origin xyz="${xpos} ${ypos} ${0}" rpy="0 0 1.57"/>
-        </joint>
-      </xacro:unless>
-  </xacro:macro>
-  <xacro:wheel prefix="first_wheel_left" xpos="0" ypos="${0}" wheel_num="1" />
-  <xacro:wheel prefix="first_wheel_right" xpos="${0}" ypos="-${0}" wheel_num="1" />
-  <!-- Except with the first wheels (steering), from second to fourth wheels are shaft's children-->
-  <xacro:wheel prefix="second_wheel_left" xpos="${base_width/2 + wheel_ygap}" ypos="${0}" wheel_num="2" />
-  <xacro:wheel prefix="second_wheel_right" xpos="-${base_width/2 + wheel_ygap}" ypos="${0}" wheel_num="2" />
-  <xacro:wheel prefix="third_wheel_left" xpos="${base_width/2 + wheel_ygap}" ypos="${0}" wheel_num="3" />
-  <xacro:wheel prefix="third_wheel_right" xpos="-${base_width/2 + wheel_ygap}" ypos="-${0}" wheel_num="3" />
-  <xacro:wheel prefix="fourth_wheel_left" xpos="${base_width/2 + wheel_ygap}" ypos="${0}" wheel_num="4" />
-  <xacro:wheel prefix="fourth_wheel_right" xpos="-${base_width/2 + wheel_ygap}" ypos="-${0}" wheel_num="4" />
+  <xacro:wheel prefix="drivewhl_l" x_reflect="-1" y_reflect="1" />
+  <xacro:wheel prefix="drivewhl_r" x_reflect="-1" y_reflect="-1" />
+  <link name="front_caster">
+    <visual>
+      <geometry>
+        <sphere radius="${(wheel_radius+wheel_zoff-(base_height/2))}"/>
+      </geometry>
+      <material name="Cyan">
+        <color rgba="0 1.0 1.0 1.0"/>
+      </material>
+    </visual>
+    <collision>
+      <origin xyz="0 0 0" rpy="0 0 0"/>
+      <geometry>
+        <sphere radius="${(wheel_radius+wheel_zoff-(base_height/2))}"/>
+      </geometry>
+    </collision>
+    <xacro:sphere_inertia m="0.5" r="${(wheel_radius+wheel_zoff-(base_height/2))}"/>
+  </link>
+  <joint name="caster_joint" type="fixed">
+    <parent link="base_link"/>
+    <child link="front_caster"/>
+    <origin xyz="${caster_xoff} 0.0 ${-(base_height/2)}" rpy="0 0 0"/>
+  </joint>
+  <link name="imu_link">
+    <visual>
+      <geometry>
+        <box size="0.1 0.1 0.1"/>
+      </geometry>
+    </visual>
+    <collision>
+      <geometry>
+        <box size="0.1 0.1 0.1"/>
+      </geometry>
+    </collision>
+    <xacro:box_inertia m="0.1" w="0.1" d="0.1" h="0.1"/>
+  </link>
+  <joint name="imu_joint" type="fixed">
+    <parent link="base_link"/>
+    <child link="imu_link"/>
+    <origin xyz="0 0 0.01"/>
+  </joint>
+  <gazebo reference="imu_link">
+    <sensor name="imu_sensor" type="imu">
+      <plugin filename="libgazebo_ros_imu_sensor.so" name="imu_plugin">
+        <ros>
+          <!-- <namespace>/demo</namespace> -->
+          <remapping>~/out:=imu</remapping>
+        </ros>
+        <initial_orientation_as_reference>false</initial_orientation_as_reference>
+      </plugin>
+      <always_on>true</always_on>
+      <update_rate>100</update_rate>
+      <visualize>true</visualize>
+     <imu>
+     	<angular_velocity>
+     	  <x>
+     	    <noise type="gaussian">
+              <mean>0.0</mean>
+              <stddev>2e-4</stddev>
+              <bias_mean>0.0000075</bias_mean>
+              <bias_stddev>0.0000008</bias_stddev>
+            </noise>
+          </x>
+          <y>
+            <noise type="gaussian">
+              <mean>0.0</mean>
+              <stddev>2e-4</stddev>
+              <bias_mean>0.0000075</bias_mean>
+              <bias_stddev>0.0000008</bias_stddev>
+            </noise>
+          </y>
+          <z>
+            <noise type="gaussian">
+              <mean>0.0</mean>
+              <stddev>2e-4</stddev>
+              <bias_mean>0.0000075</bias_mean>
+              <bias_stddev>0.0000008</bias_stddev>
+            </noise>
+          </z>
+        </angular_velocity>
+        <linear_acceleration>
+          <x>
+            <noise type="gaussian">
+              <mean>0.0</mean>
+              <stddev>1.7e-2</stddev>
+              <bias_mean>0.1</bias_mean>
+              <bias_stddev>0.001</bias_stddev>
+            </noise>
+          </x>
+          <y>
+            <noise type="gaussian">
+              <mean>0.0</mean>
+              <stddev>1.7e-2</stddev>
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